File: pcb/receiver-4x.sch (EAGLE design)
At the start: 24 parts, among them IC1 MAX3095CEE

Commit message: Receiver 4x: Rev B design
Parts:
- JP1, JP2, JP3, JP4: device SparkFun-Connectors:M03-SCREW-5MM -> LEDscape:M03SCREW-DETACH
Changed lines of the file:
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@@
 <part name="U$1" library="LEDscape" deviceset="RJ45_2X1" device=""/>
 <part name="GND2" library="SparkFun-Aesthetics" deviceset="GND" device=""/>
-<part name="JP1" library="SparkFun-Connectors" deviceset="M03" device="-SCREW-5MM"/>
-<part name="JP2" library="SparkFun-Connectors" deviceset="M03" device="-SCREW-5MM"/>
-<part name="JP3" library="SparkFun-Connectors" deviceset="M03" device="-SCREW-5MM"/>
-<part name="JP4" library="SparkFun-Connectors" deviceset="M03" device="-SCREW-5MM"/>
+<part name="JP1" library="LEDscape" deviceset="M03" device="SCREW-DETACH"/>
+<part name="JP2" library="LEDscape" deviceset="M03" device="SCREW-DETACH"/>
+<part name="JP3" library="LEDscape" deviceset="M03" device="SCREW-DETACH"/>
+<part name="JP4" library="LEDscape" deviceset="M03" device="SCREW-DETACH"/>
 <part name="R1" library="adafruit" deviceset="R-US_" device="R0603" value="100"/>
 <part name="R2" library="adafruit" deviceset="R-US_" device="R0603" value="100"/>
